Commit message: nicla camera and tof integration

File: dagana_urdf/urdf/dagana.urdf.xacro (robot description, xacro)
@@ -2,7 +2,4 @@
 <robot xmlns:xacro="http://ros.org/wiki/xacro" name="dagana">
 <xacro:include filename="$(find dagana_urdf)/urdf/dagana_macro.urdf.xacro" />
-<material name="dark_grey">
-	<color rgba="0.2 0.2 0.2 1"/>
-</material>
 <link name="world"/>
 <joint name="virtualFixed" type="fixed">

File: dagana_urdf/urdf/dagana_macro.urdf.xacro (robot description, xacro)
@@ -1,9 +1,6 @@
 <?xml version="1.0"?>
 <robot xmlns:xacro="http://ros.org/wiki/xacro">
+<xacro:include filename="$(find dagana_urdf)/urdf/config/dagana_config.urdf.xacro" />
 <xacro:macro name="dagana_gripper" params="name joint_type parent_link *origin">
-    <xacro:property name="mmTom" value="1e-3" />
-    <xacro:property name="mm2Tom2" value="1e-6" />
-    <xacro:property name="PI_2" value="1.57079632679" />
-    <xacro:property name="PI" value="3.14159265359" />
     <joint name="${name}_mount_joint" type="fixed">
         <xacro:insert_block name="origin"/>
@@ -27,5 +24,5 @@
                 <mesh filename="package://dagana_urdf/meshes/dg0001-simplified.stl" scale="${mmTom} ${mmTom} ${mmTom}" />
             </geometry>
-            <material name="dark_grey"/>
+            <material name="dagana_dark_grey"/>
         </visual>
         <collision>
@@ -34,5 +31,4 @@
                 <mesh filename="package://dagana_urdf/meshes/dg0001-simplified_v2.stl" scale="${mmTom} ${mmTom} ${mmTom}" />
             </geometry>
-            <material name="dark_grey"/>
         </collision>
     </link>
@@ -60,5 +56,5 @@
                 <mesh filename="package://dagana_urdf/meshes/dg0002.stl" scale="${mmTom} ${mmTom} ${mmTom}" />
             </geometry>
-            <material name="dark_grey"/>
+            <material name="dagana_dark_grey"/>
         </visual>
         <collision>
@@ -67,5 +63,4 @@
                 <mesh filename="package://dagana_urdf/meshes/dg0002-ch.stl" scale="${mmTom} ${mmTom} ${mmTom}" />
             </geometry>
-            <material name="dark_grey"/>
         </collision>
     </link>
@@ -77,4 +72,85 @@
     </joint>
     <link name="${name}_tcp"></link>
+    <gazebo reference="${name}_bottom_link">
+        <material>Gazebo/DarkGrey</material>
+    </gazebo>
+    <gazebo reference="${name}_top_link">
+        <material>Gazebo/DarkGrey</material>
+    </gazebo>
+    <!-- NICLA PART -->
+    <xacro:if value="${NICLA_CAMERA}">
+        <link name="nicla_camera"></link>
+        <joint name="base_to_camera" type="fixed">
+            <origin xyz="0.0000044 -0.0234997 0.1039715" rpy="0 ${-PI/2} ${-PI/2}"/>
+            <parent link="${name}_top_link"/>
+            <child link="nicla_camera"/>
+        </joint>
+        <!-- gazebo simulated camera -->
+        <gazebo reference="nicla_camera">
+        <sensor type="camera" name="camera1">
+        <update_rate>30.0</update_rate>
+        <camera name="head">
+            <horizontal_fov>0.69813</horizontal_fov>  <!-- 80deg 1.39626rad-->
+            <image>
+                <width>1616</width>
+                <height>1232</height>
+                <format>R8G8B8</format>
+            </image>
+            <clip>
+                <near>0.1</near>
+                <far>100</far>
+          </clip>
+        </camera>
+        <plugin name="gazebo_ros_nicla_camera_controller" filename="libgazebo_ros_camera.so">
+            <alwaysOn>true</alwaysOn>
+            <updateRate>0.0</updateRate>
+            <cameraName>dagana/nicla_camera</cameraName>
+            <imageTopicName>image_raw</imageTopicName>
+            <cameraInfoTopicName>camera_info</cameraInfoTopicName>
+            <frameName>nicla_camera</frameName>
+        </plugin>
+        </sensor>
+        </gazebo>
+    </xacro:if>
+    <xacro:if value="${NICLA_TOF}">
+        <link name="nicla_tof"></link>
+        <joint name="base_to_tof" type="fixed">
+            <origin xyz="0.0000044 -0.0234997 0.1039715" rpy="0 ${-PI/2} 0"/>
+            <parent link="${name}_top_link"/>
+            <child link="nicla_tof"/>
+        </joint>
+        <!-- gazebo simulated tof -->
+        <gazebo reference="nicla_tof">
+        <sensor type="ray" name="nicla_tof">
+        <pose>0 0 0 0 0 0</pose>
+        <visualize>${nicla_tof_visualize}</visualize>
+        <update_rate>60</update_rate>
+        <ray>
+            <scan>
+            <horizontal>
+                <samples>1</samples>
+                <resolution>1</resolution>
+                <min_angle>0</min_angle>
+                <max_angle>0</max_angle>
+            </horizontal>
+            </scan>
+            <range>
+            <min>0.04</min>
+            <max>3</max>
+            <resolution>0.03</resolution>
+            </range>
+            <!-- <noise>
+                <type>gaussian</type>
+                <mean>0.0</mean>
+                <stddev>0.01</stddev>
+            </noise> -->
+        </ray>
+        <plugin name="gazebo_ros_nicla_tof_controller" filename="libgazebo_ros_laser.so">
+            <topicName>/dagana/nicla_tof</topicName>
+            <frameName>nicla_tof</frameName>
+        </plugin>
+        </sensor>
+        </gazebo>
+    </xacro:if>
 </xacro:macro>
 </robot>
