Commit message: upd formwork weights

File: dagana_urdf/urdf/dagana_macro.urdf.xacro (robot description, xacro)
@@ -37,5 +37,5 @@
             <inertial>
                 <origin xyz="${-6.2068321e+00*mmTom} ${-1.1480379e+01*mmTom}  ${4.7628197e+01*mmTom}" rpy="0 0 0"/>
-                <mass value="1.464"/>
+                <mass value="1.548"/>
                 <inertia ixx="${2.8611741e+03*mm2Tom2}"
                         ixy="${-2.7536524e+00*mm2Tom2}"
@@ -107,5 +107,5 @@
             <inertial>
                 <origin xyz="${2.5812008e+01*mmTom} ${2.5751001e+00*mmTom} ${-4.9454259e+00*mmTom}" rpy="0 0 0"/>
-                <mass value="1.8562763e-01"/>
+                <mass value="2.18e-01"/>
                 <inertia ixx="${4.5712825e+02*mm2Tom2}"
                         ixy="${-1.1939252e+01*mm2Tom2}"
@@ -169,5 +169,5 @@
             <inertial>
                 <origin xyz="0.0 ${-5.0362316e+00*mmTom} ${4.8400486e+01*mmTom}" rpy="0 0 0"/>
-                <mass value="4.6341578e-01"/>
+                <mass value="4.26e-01"/>
                 <inertia ixx="${5.6823263e+02*mm2Tom2}"
                         ixy="${0.0*mm2Tom2}"
@@ -194,5 +194,5 @@
             <inertial>
                 <origin xyz="0.0 ${-3.3025449e+00*mmTom} ${5.2167268e+01*mmTom}" rpy="0 0 0"/>
-                <mass value="3.9065902e-01"/>
+                <mass value="3.52e-01"/>
                 <inertia ixx="${5.2459269e+02*mm2Tom2}"
                         ixy="${0.0*mm2Tom2}"

Commit message: add simplified and ch meshes for concert jaws

File: dagana_urdf/urdf/dagana_macro.urdf.xacro (robot description, xacro)
@@ -48,12 +48,12 @@
                 <origin xyz="0 0 0" rpy="0 0 0" />
                 <geometry>
-                    <mesh filename="package://dagana_urdf/meshes/mesh_dagana-base.stl" scale="${mmTom} ${mmTom} ${mmTom}" />
-                </geometry>
-                <material name="dagana_dark_grey"/>
-            </visual>
-            <collision>
-                <origin xyz="0 0 0" rpy="0 0 0" />
-                <geometry>
-                    <mesh filename="package://dagana_urdf/meshes/mesh_dagana-base.stl" scale="${mmTom} ${mmTom} ${mmTom}" />
+                    <mesh filename="package://dagana_urdf/meshes/mesh_dagana-base_simple.stl" scale="${mmTom} ${mmTom} ${mmTom}" />
+                </geometry>
+                <material name="dagana_dark_grey"/>
+            </visual>
+            <collision>
+                <origin xyz="0 0 0" rpy="0 0 0" />
+                <geometry>
+                    <mesh filename="package://dagana_urdf/meshes/mesh_dagana-base_ch.stl" scale="${mmTom} ${mmTom} ${mmTom}" />
                 </geometry>
             </collision>
@@ -118,12 +118,12 @@
                 <origin xyz="0 0 0" rpy="0 0 0" />
                 <geometry>
-                    <mesh filename="package://dagana_urdf/meshes/mesh_dagana-link.stl" scale="${mmTom} ${mmTom} ${mmTom}" />
-                </geometry>
-                <material name="dagana_dark_grey"/>
-            </visual>
-            <collision>
-                <origin xyz="0 0 0" rpy="0 0 0" />
-                <geometry>
-                    <mesh filename="package://dagana_urdf/meshes/mesh_dagana-link.stl" scale="${mmTom} ${mmTom} ${mmTom}" />
+                    <mesh filename="package://dagana_urdf/meshes/mesh_dagana-link_simple.stl" scale="${mmTom} ${mmTom} ${mmTom}" />
+                </geometry>
+                <material name="dagana_dark_grey"/>
+            </visual>
+            <collision>
+                <origin xyz="0 0 0" rpy="0 0 0" />
+                <geometry>
+                    <mesh filename="package://dagana_urdf/meshes/mesh_dagana-link_ch.stl" scale="${mmTom} ${mmTom} ${mmTom}" />
                 </geometry>
             </collision>
@@ -187,5 +187,5 @@
                 <origin xyz="0 0 0" rpy="0 0 0" />
                 <geometry>
-                    <mesh filename="package://dagana_urdf/meshes/mesh_formwork-base.stl" scale="${mmTom} ${mmTom} ${mmTom}" />
+                    <mesh filename="package://dagana_urdf/meshes/mesh_formwork-base_ch.stl" scale="${mmTom} ${mmTom} ${mmTom}" />
                 </geometry>
             </collision>
@@ -212,5 +212,5 @@
                 <origin xyz="0 0 0" rpy="0 0 0" />
                 <geometry>
-                    <mesh filename="package://dagana_urdf/meshes/mesh_formwork-thumb.stl" scale="${mmTom} ${mmTom} ${mmTom}" />
+                    <mesh filename="package://dagana_urdf/meshes/mesh_formwork-thumb_ch.stl" scale="${mmTom} ${mmTom} ${mmTom}" />
                 </geometry>
             </collision>
@@ -232,12 +232,12 @@
                 <origin xyz="0 0 0" rpy="0 0 0" />
                 <geometry>
-                    <mesh filename="package://dagana_urdf/meshes/mesh_tube-thumb.stl" scale="${mmTom} ${mmTom} ${mmTom}" />
-                </geometry>
-                <material name="dagana_dark_grey"/>
-            </visual>
-            <collision>
-                <origin xyz="0 0 0" rpy="0 0 0" />
-                <geometry>
-                    <mesh filename="package://dagana_urdf/meshes/mesh_tube-thumb.stl" scale="${mmTom} ${mmTom} ${mmTom}" />
+                    <mesh filename="package://dagana_urdf/meshes/mesh_tube-thumb_simple.stl" scale="${mmTom} ${mmTom} ${mmTom}" />
+                </geometry>
+                <material name="dagana_dark_grey"/>
+            </visual>
+            <collision>
+                <origin xyz="0 0 0" rpy="0 0 0" />
+                <geometry>
+                    <mesh filename="package://dagana_urdf/meshes/mesh_tube-thumb_ch.stl" scale="${mmTom} ${mmTom} ${mmTom}" />
                 </geometry>
             </collision>
@@ -257,12 +257,12 @@
                 <origin xyz="0 0 0" rpy="0 0 0" />
                 <geometry>
-                    <mesh filename="package://dagana_urdf/meshes/mesh_tube-base.stl" scale="${mmTom} ${mmTom} ${mmTom}" />
-                </geometry>
-                <material name="dagana_dark_grey"/>
-            </visual>
-            <collision>
-                <origin xyz="0 0 0" rpy="0 0 0" />
-                <geometry>
-                    <mesh filename="package://dagana_urdf/meshes/mesh_tube-base.stl" scale="${mmTom} ${mmTom} ${mmTom}" />
+                    <mesh filename="package://dagana_urdf/meshes/mesh_tube-base_simple.stl" scale="${mmTom} ${mmTom} ${mmTom}" />
+                </geometry>
+                <material name="dagana_dark_grey"/>
+            </visual>
+            <collision>
+                <origin xyz="0 0 0" rpy="0 0 0" />
+                <geometry>
+                    <mesh filename="package://dagana_urdf/meshes/mesh_tube-base_ch.stl" scale="${mmTom} ${mmTom} ${mmTom}" />
                 </geometry>
             </collision>

Commit message: tcp shifted a bit to the fixed part

File: dagana_urdf/urdf/dagana_macro.urdf.xacro (robot description, xacro)
@@ -67,5 +67,6 @@
     <!-- Manually put to have a transform in a "good" grasping spot-->
     <joint name="${name}_tcp_joint" type="fixed">
-        <origin xyz="0 -0.05 0.15" rpy="0 0 0"/>
+        <!-- <origin xyz="0 -0.05 0.15" rpy="0 0 0"/> -->
+        <origin xyz="0 -0.04 0.17" rpy="0 0 0"/>
         <parent link="${name}_top_link"/>
         <child link="${name}_tcp"/>

Commit message: sorry for playing with tcp

File: dagana_urdf/urdf/dagana_macro.urdf.xacro (robot description, xacro)
@@ -155,5 +155,5 @@
     <joint name="${name}_tcp_joint" type="fixed">
         <xacro:if value="${DAGANA_CLAWS_TYPE == 'centauro_claws'}">
-            <origin xyz="0 -0.04 0.17" rpy="0 0 0"/>
+            <origin xyz="0 -0.04 0.16" rpy="0 0 0"/>
         </xacro:if>
         <xacro:if value="${DAGANA_CLAWS_TYPE == 'concert_formwork_claws' or DAGANA_CLAWS_TYPE == 'concert_tube_claws'}">

Commit message: joint limit so in simulation it stops

File: dagana_urdf/urdf/dagana_macro.urdf.xacro (robot description, xacro)
@@ -75,5 +75,5 @@
             <child link="${name}_bottom_link"/>
             <axis xyz="-1 0 0"/>
-            <limit effort="1000" lower="-1.5" upper="1.3" velocity="10.0"/>
+            <limit effort="1000" lower="-0.1" upper="1.3" velocity="10.0"/>
         </joint>
     </xacro:if>

Commit message: option for separated palms

File: dagana_urdf/urdf/dagana_macro.urdf.xacro (robot description, xacro)
@@ -34,4 +34,29 @@
             </collision>
         </xacro:if>
+        <xacro:if value="${DAGANA_CLAWS_TYPE == 'centauro_claws_palm_separated'}">
+            <inertial>
+                <origin xyz="${-6.3562154e+00*mmTom} ${-6.0265532e+00*mmTom}  ${6.0068288e+01*mmTom}" rpy="0 0 0"/>
+                <mass value="1.7432400"/>
+                <inertia ixx="${5.0510328e+03*mm2Tom2}"
+                        ixy="${-2.5264216e+02*mm2Tom2}"
+                        ixz="${-1.2103013e+02*mm2Tom2}"
+                        iyy="${4.7944612e+03*mm2Tom2}"
+                        iyz="${-7.3917704e+02*mm2Tom2}"
+                        izz="${3.1156997e+03*mm2Tom2}" />
+            </inertial>
+            <visual>
+                <origin xyz="0 0 0" rpy="0 0 0" />
+                <geometry>
+                    <mesh filename="package://dagana_urdf/meshes/dg0001-simplified_v2_bottom.stl" scale="${mmTom} ${mmTom} ${mmTom}" />
+                </geometry>
+                <material name="dagana_dark_grey"/>
+            </visual>
+            <collision>
+                <origin xyz="0 0 0" rpy="0 0 0" />
+                <geometry>
+                    <mesh filename="package://dagana_urdf/meshes/dg0001-simplified_v2_bottom.stl" scale="${mmTom} ${mmTom} ${mmTom}" />
+                </geometry>
+            </collision>
+        </xacro:if>
         <xacro:if value="${DAGANA_CLAWS_TYPE == 'concert_formwork_claws' or DAGANA_CLAWS_TYPE == 'concert_tube_claws'}">
             <inertial>
@@ -60,4 +85,26 @@
         </xacro:if>
     </link>
+    <xacro:if value="${DAGANA_CLAWS_TYPE == 'centauro_claws_palm_separated'}">
+        <joint name="${name}_top_link_palm_fixed_joint" type="fixed" dont_collapse="true">
+            <origin xyz="0 0 0" rpy="0 0 0"/>
+            <parent link="${name}_top_link"/>
+            <child link="${name}_top_link_palm"/>
+        </joint>
+        <link name="${name}_top_link_palm">
+            <visual>
+                <origin xyz="0 0 0" rpy="0 0 0" />
+                <geometry>
+                    <mesh filename="package://dagana_urdf/meshes/dg0001-simplified_v2_palm.stl" scale="${mmTom} ${mmTom} ${mmTom}" />
+                </geometry>
+                <material name="dagana_dark_grey"/>
+            </visual>
+            <collision>
+                <origin xyz="0 0 0" rpy="0 0 0" />
+                <geometry>
+                    <mesh filename="package://dagana_urdf/meshes/dg0001-simplified_v2_palm.stl" scale="${mmTom} ${mmTom} ${mmTom}" />
+                </geometry>
+            </collision>
+        </link>
+    </xacro:if>
     <xacro:if value="${DAGANA_CLAWS_TYPE == 'concert_formwork_claws' or DAGANA_CLAWS_TYPE == 'concert_tube_claws'}">
         <joint name="${name}_claw_joint" type="${joint_type}">
@@ -69,5 +116,5 @@
         </joint>
     </xacro:if>
-    <xacro:if value="${DAGANA_CLAWS_TYPE == 'centauro_claws'}">
+    <xacro:if value="${DAGANA_CLAWS_TYPE == 'centauro_claws' or DAGANA_CLAWS_TYPE == 'centauro_claws_palm_separated'}">
         <joint name="${name}_claw_joint" type="${joint_type}">
             <origin xyz="${0.0*mmTom} ${-28.00*mmTom} ${50.25*mmTom}" rpy="${PI_2} 0 ${PI}"/>
@@ -104,4 +151,29 @@
             </collision>
         </xacro:if>
+        <xacro:if value="${DAGANA_CLAWS_TYPE == 'centauro_claws_palm_separated'}">
+            <inertial>
+                <origin xyz="0 ${6.9644767e+01*mmTom} 0" rpy="0 0 0"/>
+                <mass value="4.6117745e-01"/>
+                <inertia iyy="${9.3855569e+02*mm2Tom2}"
+                        iyz="${-2.6445200e+02*mm2Tom2}"
+                        ixy="${7.1346830e+01*mm2Tom2}"
+                        izz="${1.9472731e+03*mm2Tom2}"
+                        ixz="${2.5290650e+00*mm2Tom2}"
+                        ixx="${1.4726991e+03*mm2Tom2}" />
+            </inertial>
+            <visual>
+                <origin xyz="0 0 0" rpy="0 0 0" />
+                <geometry>
+                    <mesh filename="package://dagana_urdf/meshes/dg0002-ch-bottom.stl" scale="${mmTom} ${mmTom} ${mmTom}" />
+                </geometry>
+                <material name="dagana_dark_grey"/>
+            </visual>
+            <collision>
+                <origin xyz="0 0 0" rpy="0 0 0" />
+                <geometry>
+                    <mesh filename="package://dagana_urdf/meshes/dg0002-ch-bottom.stl" scale="${mmTom} ${mmTom} ${mmTom}" />
+                </geometry>
+            </collision>
+        </xacro:if>
         <xacro:if value="${DAGANA_CLAWS_TYPE == 'concert_formwork_claws' or DAGANA_CLAWS_TYPE == 'concert_tube_claws'}">
             <inertial>
@@ -130,4 +202,26 @@
         </xacro:if>
     </link>
+    <xacro:if value="${DAGANA_CLAWS_TYPE == 'centauro_claws_palm_separated'}">
+        <joint name="${name}_claw_palm_fixed_joint" type="fixed" dont_collapse="true">
+            <origin xyz="0 0 0" rpy="0 0 0"/>
+            <parent link="${name}_bottom_link"/>
+            <child link="${name}_bottom_link_palm"/>
+        </joint>
+        <link name="${name}_bottom_link_palm">
+            <visual>
+                <origin xyz="0 0 0" rpy="0 0 0" />
+                <geometry>
+                    <mesh filename="package://dagana_urdf/meshes/dg0002-ch-palm.stl" scale="${mmTom} ${mmTom} ${mmTom}" />
+                </geometry>
+                <material name="dagana_dark_grey"/>
+            </visual>
+            <collision>
+                <origin xyz="0 0 0" rpy="0 0 0" />
+                <geometry>
+                    <mesh filename="package://dagana_urdf/meshes/dg0002-ch-palm.stl" scale="${mmTom} ${mmTom} ${mmTom}" />
+                </geometry>
+            </collision>
+        </link>
+    </xacro:if>
     <xacro:if value="${GAZEBO_URDF}">
         <gazebo reference="${name}_bottom_link">

Commit message: better separated palms

File: dagana_urdf/urdf/dagana_macro.urdf.xacro (robot description, xacro)
@@ -35,4 +35,5 @@
         </xacro:if>
         <xacro:if value="${DAGANA_CLAWS_TYPE == 'centauro_claws_palm_separated'}">
+            <!-- TODO this is the inertial of the entire piece (ABC), it should be divided among the different pieces -->
             <inertial>
                 <origin xyz="${-6.3562154e+00*mmTom} ${-6.0265532e+00*mmTom}  ${6.0068288e+01*mmTom}" rpy="0 0 0"/>
@@ -48,12 +49,12 @@
                 <origin xyz="0 0 0" rpy="0 0 0" />
                 <geometry>
-                    <mesh filename="package://dagana_urdf/meshes/dg0001-simplified_v2_bottom.stl" scale="${mmTom} ${mmTom} ${mmTom}" />
-                </geometry>
-                <material name="dagana_dark_grey"/>
-            </visual>
-            <collision>
-                <origin xyz="0 0 0" rpy="0 0 0" />
-                <geometry>
-                    <mesh filename="package://dagana_urdf/meshes/dg0001-simplified_v2_bottom.stl" scale="${mmTom} ${mmTom} ${mmTom}" />
+                    <mesh filename="package://dagana_urdf/meshes/dagana_fixed_A.stl" scale="${mmTom} ${mmTom} ${mmTom}" />
+                </geometry>
+                <material name="dagana_dark_grey"/>
+            </visual>
+            <collision>
+                <origin xyz="0 0 0" rpy="0 0 0" />
+                <geometry>
+                    <mesh filename="package://dagana_urdf/meshes/dagana_fixed_A_simple.stl" scale="${mmTom} ${mmTom} ${mmTom}" />
                 </geometry>
             </collision>
@@ -86,21 +87,41 @@
     </link>
     <xacro:if value="${DAGANA_CLAWS_TYPE == 'centauro_claws_palm_separated'}">
-        <joint name="${name}_top_link_palm_fixed_joint" type="fixed" dont_collapse="true">
+        <joint name="${name}_fixed_A_B_fixed_joint" type="fixed" dont_collapse="true">
             <origin xyz="0 0 0" rpy="0 0 0"/>
             <parent link="${name}_top_link"/>
-            <child link="${name}_top_link_palm"/>
-        </joint>
-        <link name="${name}_top_link_palm">
-            <visual>
-                <origin xyz="0 0 0" rpy="0 0 0" />
-                <geometry>
-                    <mesh filename="package://dagana_urdf/meshes/dg0001-simplified_v2_palm.stl" scale="${mmTom} ${mmTom} ${mmTom}" />
-                </geometry>
-                <material name="dagana_dark_grey"/>
-            </visual>
-            <collision>
-                <origin xyz="0 0 0" rpy="0 0 0" />
-                <geometry>
-                    <mesh filename="package://dagana_urdf/meshes/dg0001-simplified_v2_palm.stl" scale="${mmTom} ${mmTom} ${mmTom}" />
+            <child link="${name}_fixed_B"/>
+        </joint>
+        <link name="${name}_fixed_B">
+            <visual>
+                <origin xyz="0 0 0" rpy="0 0 0" />
+                <geometry>
+                    <mesh filename="package://dagana_urdf/meshes/dagana_fixed_B.stl" scale="${mmTom} ${mmTom} ${mmTom}" />
+                </geometry>
+                <material name="dagana_dark_grey"/>
+            </visual>
+            <collision>
+                <origin xyz="0 0 0" rpy="0 0 0" />
+                <geometry>
+                    <mesh filename="package://dagana_urdf/meshes/dagana_fixed_B_simple.stl" scale="${mmTom} ${mmTom} ${mmTom}" />
+                </geometry>
+            </collision>
+        </link>
+        <joint name="${name}_fixed_B_C_fixed_joint" type="fixed" dont_collapse="true">
+            <origin xyz="0 0 0" rpy="0 0 0"/>
+            <parent link="${name}_fixed_B"/>
+            <child link="${name}_fixed_C"/>
+        </joint>
+        <link name="${name}_fixed_C">
+            <visual>
+                <origin xyz="0 0 0" rpy="0 0 0" />
+                <geometry>
+                    <mesh filename="package://dagana_urdf/meshes/dagana_fixed_C.stl" scale="${mmTom} ${mmTom} ${mmTom}" />
+                </geometry>
+                <material name="dagana_dark_grey"/>
+            </visual>
+            <collision>
+                <origin xyz="0 0 0" rpy="0 0 0" />
+                <geometry>
+                    <mesh filename="package://dagana_urdf/meshes/dagana_fixed_C_simple.stl" scale="${mmTom} ${mmTom} ${mmTom}" />
                 </geometry>
             </collision>
@@ -165,12 +186,12 @@
                 <origin xyz="0 0 0" rpy="0 0 0" />
                 <geometry>
-                    <mesh filename="package://dagana_urdf/meshes/dg0002-ch-bottom.stl" scale="${mmTom} ${mmTom} ${mmTom}" />
-                </geometry>
-                <material name="dagana_dark_grey"/>
-            </visual>
-            <collision>
-                <origin xyz="0 0 0" rpy="0 0 0" />
-                <geometry>
-                    <mesh filename="package://dagana_urdf/meshes/dg0002-ch-bottom.stl" scale="${mmTom} ${mmTom} ${mmTom}" />
+                    <mesh filename="package://dagana_urdf/meshes/dagana_claw_A.stl" scale="${mmTom} ${mmTom} ${mmTom}" />
+                </geometry>
+                <material name="dagana_dark_grey"/>
+            </visual>
+            <collision>
+                <origin xyz="0 0 0" rpy="0 0 0" />
+                <geometry>
+                    <mesh filename="package://dagana_urdf/meshes/dagana_claw_A_simple.stl" scale="${mmTom} ${mmTom} ${mmTom}" />
                 </geometry>
             </collision>
@@ -203,21 +224,21 @@
     </link>
     <xacro:if value="${DAGANA_CLAWS_TYPE == 'centauro_claws_palm_separated'}">
-        <joint name="${name}_claw_palm_fixed_joint" type="fixed" dont_collapse="true">
+        <joint name="${name}_claw_A_B_fixed_joint" type="fixed" dont_collapse="true">
             <origin xyz="0 0 0" rpy="0 0 0"/>
             <parent link="${name}_bottom_link"/>
-            <child link="${name}_bottom_link_palm"/>
-        </joint>
-        <link name="${name}_bottom_link_palm">
-            <visual>
-                <origin xyz="0 0 0" rpy="0 0 0" />
-                <geometry>
-                    <mesh filename="package://dagana_urdf/meshes/dg0002-ch-palm.stl" scale="${mmTom} ${mmTom} ${mmTom}" />
-                </geometry>
-                <material name="dagana_dark_grey"/>
-            </visual>
-            <collision>
-                <origin xyz="0 0 0" rpy="0 0 0" />
-                <geometry>
-                    <mesh filename="package://dagana_urdf/meshes/dg0002-ch-palm.stl" scale="${mmTom} ${mmTom} ${mmTom}" />
+            <child link="${name}_claw_B"/>
+        </joint>
+        <link name="${name}_claw_B">
+            <visual>
+                <origin xyz="0 0 0" rpy="0 0 0" />
+                <geometry>
+                    <mesh filename="package://dagana_urdf/meshes/dagana_claw_B.stl" scale="${mmTom} ${mmTom} ${mmTom}" />
+                </geometry>
+                <material name="dagana_dark_grey"/>
+            </visual>
+            <collision>
+                <origin xyz="0 0 0" rpy="0 0 0" />
+                <geometry>
+                    <mesh filename="package://dagana_urdf/meshes/dagana_claw_B_simple.stl" scale="${mmTom} ${mmTom} ${mmTom}" />
                 </geometry>
             </collision>
