Commit message: niclabox on dedicated repo

File: dagana_urdf/urdf/config/dagana_config.urdf.xacro (robot description, xacro)
@@ -1,5 +1,5 @@
 <?xml version="1.0"?>
 <robot xmlns:xacro="http://ros.org/wiki/xacro" name="dagana">
-<xacro:arg name="nicla_camera" default="true"/>
+<xacro:arg name="nicla_camera" default="false"/>
 <xacro:arg name="nicla_tof" default="true"/>
 <xacro:arg name="nicla_tof_visualize" default="true"/>

File: dagana_urdf/urdf/dagana_macro.urdf.xacro (robot description, xacro)
@@ -80,76 +80,8 @@
     <!-- NICLA PART -->
     <xacro:if value="${NICLA_CAMERA}">
-        <link name="nicla_camera"></link>
-        <joint name="base_to_camera" type="fixed">
+    	<xacro:include filename="$(find niclabox)/urdf/nicla_macro.urdf.xacro" />
+		<xacro:nicla_box parent_link="${name}_top_link">
             <origin xyz="0.0000044 -0.0234997 0.1039715" rpy="0 ${-PI/2} ${-PI/2}"/>
-            <parent link="${name}_top_link"/>
-            <child link="nicla_camera"/>
-        </joint>
-        <!-- gazebo simulated camera -->
-        <gazebo reference="nicla_camera">
-        <sensor type="camera" name="camera1">
-        <update_rate>30.0</update_rate>
-        <camera name="head">
-            <horizontal_fov>0.69813</horizontal_fov>  <!-- 80deg 1.39626rad-->
-            <image>
-                <width>1616</width>
-                <height>1232</height>
-                <format>R8G8B8</format>
-            </image>
-            <clip>
-                <near>0.1</near>
-                <far>100</far>
-          </clip>
-        </camera>
-        <plugin name="gazebo_ros_nicla_camera_controller" filename="libgazebo_ros_camera.so">
-            <alwaysOn>true</alwaysOn>
-            <updateRate>0.0</updateRate>
-            <cameraName>dagana/nicla_camera</cameraName>
-            <imageTopicName>image_raw</imageTopicName>
-            <cameraInfoTopicName>camera_info</cameraInfoTopicName>
-            <frameName>nicla_camera</frameName>
-        </plugin>
-        </sensor>
-        </gazebo>
-    </xacro:if>
-    <xacro:if value="${NICLA_TOF}">
-        <link name="nicla_tof"></link>
-        <joint name="base_to_tof" type="fixed">
-            <origin xyz="0.0000044 -0.0234997 0.1039715" rpy="0 ${-PI/2} 0"/>
-            <parent link="${name}_top_link"/>
-            <child link="nicla_tof"/>
-        </joint>
-        <!-- gazebo simulated tof -->
-        <gazebo reference="nicla_tof">
-        <sensor type="ray" name="nicla_tof">
-        <pose>0 0 0 0 0 0</pose>
-        <visualize>${nicla_tof_visualize}</visualize>
-        <update_rate>60</update_rate>
-        <ray>
-            <scan>
-            <horizontal>
-                <samples>1</samples>
-                <resolution>1</resolution>
-                <min_angle>0</min_angle>
-                <max_angle>0</max_angle>
-            </horizontal>
-            </scan>
-            <range>
-            <min>0.04</min>
-            <max>3</max>
-            <resolution>0.03</resolution>
-            </range>
-            <!-- <noise>
-                <type>gaussian</type>
-                <mean>0.0</mean>
-                <stddev>0.01</stddev>
-            </noise> -->
-        </ray>
-        <plugin name="gazebo_ros_nicla_tof_controller" filename="libgazebo_ros_laser.so">
-            <topicName>/dagana/nicla_tof</topicName>
-            <frameName>nicla_tof</frameName>
-        </plugin>
-        </sensor>
-        </gazebo>
+		</xacro:nicla_box>
     </xacro:if>
 </xacro:macro>

Commit message: new nicla

File: dagana_urdf/urdf/config/dagana_config.urdf.xacro (robot description, xacro)
@@ -1,8 +1,10 @@
 <?xml version="1.0"?>
 <robot xmlns:xacro="http://ros.org/wiki/xacro" name="dagana">
+<xacro:arg name="nicla" default="false"/>
 <xacro:arg name="nicla_camera" default="false"/>
 <xacro:arg name="nicla_tof" default="true"/>
 <xacro:arg name="nicla_tof_visualize" default="true"/>
-<xacro:arg name="nicla_imu" default="false"/> <!-- TODO -->
+<xacro:arg name="nicla_imu" default="false"/>
+<xacro:property name="NICLA" value="$(arg nicla)" />
 <xacro:property name="NICLA_CAMERA" value="$(arg nicla_camera)" />
 <xacro:property name="NICLA_TOF" value="$(arg nicla_tof)" />

File: dagana_urdf/urdf/dagana_macro.urdf.xacro (robot description, xacro)
@@ -79,8 +79,9 @@
     </gazebo>
     <!-- NICLA PART -->
-    <xacro:if value="${NICLA_CAMERA}">
-    	<xacro:include filename="$(find niclabox)/urdf/nicla_macro.urdf.xacro" />
+    <xacro:if value="${NICLA}">
+    	<xacro:include filename="$(find nicla_vision_ros)/urdf/nicla_macro.urdf.xacro" />
 		<xacro:nicla_box parent_link="${name}_top_link">
-            <origin xyz="0.0000044 -0.0234997 0.1039715" rpy="0 ${-PI/2} ${-PI/2}"/>
+            <!-- <origin xyz="0.0000044 -0.0234997 0.1039715" rpy="0 0 ${PI}"/> THIS IS TOP LINK TO CAMERA-->
+            <origin xyz="-0.002506 -0.0157197 0.0994715" rpy="0 0 ${PI}"/>
 		</xacro:nicla_box>
     </xacro:if>

Commit message: add `dagana_claws_type` dagna macro arg

File: dagana_urdf/urdf/config/dagana_config.urdf.xacro (robot description, xacro)
@@ -6,4 +6,8 @@
 <xacro:arg name="nicla_tof_visualize" default="true"/>
 <xacro:arg name="nicla_imu" default="true"/>
+<xacro:arg name="dagana_claws_type" default="centauro_claws"/>
+<!-- dagana_claws_types: - 'centauro_claws' -->
+<!--                     - 'concert_formwork_claws' -->
+<!--                     - 'concert_tube_claws'  -->
 <xacro:property name="NICLA" value="$(arg nicla)" />
 <xacro:property name="NICLA_CAMERA" value="$(arg nicla_camera)" />
@@ -18,3 +22,4 @@
 <xacro:property name="PI_2" value="1.57079632679" />
 <xacro:property name="PI" value="3.14159265359" />
+<xacro:property name="DAGANA_CLAWS_TYPE" value="$(arg dagana_claws_type)" />
 </robot>

File: dagana_urdf/urdf/dagana_macro.urdf.xacro (robot description, xacro)
@@ -9,27 +9,79 @@
     </joint>
     <link name="${name}_top_link">
-        <inertial>
-            <origin xyz="${-6.3562154e+00*mmTom} ${-6.0265532e+00*mmTom}  ${6.0068288e+01*mmTom}" rpy="0 0 0"/>
-            <mass value="1.7432400"/>
-            <inertia ixx="${5.0510328e+03*mm2Tom2}"
-                     ixy="${-2.5264216e+02*mm2Tom2}"
-                     ixz="${-1.2103013e+02*mm2Tom2}"
-                     iyy="${4.7944612e+03*mm2Tom2}"
-                     iyz="${-7.3917704e+02*mm2Tom2}"
-                     izz="${3.1156997e+03*mm2Tom2}" />
-        </inertial>
-        <visual>
-            <origin xyz="0 0 0" rpy="0 0 0" />
-            <geometry>
-                <mesh filename="package://dagana_urdf/meshes/dg0001-simplified.stl" scale="${mmTom} ${mmTom} ${mmTom}" />
-            </geometry>
-            <material name="dagana_dark_grey"/>
-        </visual>
-        <collision>
-            <origin xyz="0 0 0" rpy="0 0 0" />
-            <geometry>
-                <mesh filename="package://dagana_urdf/meshes/dg0001-simplified_v2.stl" scale="${mmTom} ${mmTom} ${mmTom}" />
-            </geometry>
-        </collision>
+        <xacro:if value="${DAGANA_CLAWS_TYPE == 'centauro_claws'}">
+            <inertial>
+                <origin xyz="${-6.3562154e+00*mmTom} ${-6.0265532e+00*mmTom}  ${6.0068288e+01*mmTom}" rpy="0 0 0"/>
+                <mass value="1.7432400"/>
+                <inertia ixx="${5.0510328e+03*mm2Tom2}"
+                        ixy="${-2.5264216e+02*mm2Tom2}"
+                        ixz="${-1.2103013e+02*mm2Tom2}"
+                        iyy="${4.7944612e+03*mm2Tom2}"
+                        iyz="${-7.3917704e+02*mm2Tom2}"
+                        izz="${3.1156997e+03*mm2Tom2}" />
+            </inertial>
+            <visual>
+                <origin xyz="0 0 0" rpy="0 0 0" />
+                <geometry>
+                    <mesh filename="package://dagana_urdf/meshes/dg0001-simplified.stl" scale="${mmTom} ${mmTom} ${mmTom}" />
+                </geometry>
+                <material name="dagana_dark_grey"/>
+            </visual>
+            <collision>
+                <origin xyz="0 0 0" rpy="0 0 0" />
+                <geometry>
+                    <mesh filename="package://dagana_urdf/meshes/dg0001-simplified_v2.stl" scale="${mmTom} ${mmTom} ${mmTom}" />
+                </geometry>
+            </collision>
+        </xacro:if>
+        <xacro:if value="${DAGANA_CLAWS_TYPE == 'concert_formwork_claws'}">
+            <inertial>
+                <origin xyz="${-6.3562154e+00*mmTom} ${-6.0265532e+00*mmTom}  ${6.0068288e+01*mmTom}" rpy="0 0 0"/>
+                <mass value="1.870"/>
+                <inertia ixx="${5.0510328e+03*mm2Tom2}"
+                        ixy="${-2.5264216e+02*mm2Tom2}"
+                        ixz="${-1.2103013e+02*mm2Tom2}"
+                        iyy="${4.7944612e+03*mm2Tom2}"
+                        iyz="${-7.3917704e+02*mm2Tom2}"
+                        izz="${3.1156997e+03*mm2Tom2}" />
+            </inertial>
+            <visual>
+                <origin xyz="0 0 0" rpy="0 0 0" />
+                <geometry>
+                    <mesh filename="package://dagana_urdf/meshes/dg0001-simplified.stl" scale="${mmTom} ${mmTom} ${mmTom}" />
+                </geometry>
+                <material name="dagana_dark_grey"/>
+            </visual>
+            <collision>
+                <origin xyz="0 0 0" rpy="0 0 0" />
+                <geometry>
+                    <mesh filename="package://dagana_urdf/meshes/dg0001-simplified_v2.stl" scale="${mmTom} ${mmTom} ${mmTom}" />
+                </geometry>
+            </collision>
+        </xacro:if>
+        <xacro:if value="${DAGANA_CLAWS_TYPE == 'concert_tube_claws'}">
+            <inertial>
+                <origin xyz="${-6.3562154e+00*mmTom} ${-6.0265532e+00*mmTom}  ${6.0068288e+01*mmTom}" rpy="0 0 0"/>
+                <mass value="1.929"/>
+                <inertia ixx="${5.0510328e+03*mm2Tom2}"
+                        ixy="${-2.5264216e+02*mm2Tom2}"
+                        ixz="${-1.2103013e+02*mm2Tom2}"
+                        iyy="${4.7944612e+03*mm2Tom2}"
+                        iyz="${-7.3917704e+02*mm2Tom2}"
+                        izz="${3.1156997e+03*mm2Tom2}" />
+            </inertial>
+            <visual>
+                <origin xyz="0 0 0" rpy="0 0 0" />
+                <geometry>
+                    <mesh filename="package://dagana_urdf/meshes/dg0001-simplified.stl" scale="${mmTom} ${mmTom} ${mmTom}" />
+                </geometry>
+                <material name="dagana_dark_grey"/>
+            </visual>
+            <collision>
+                <origin xyz="0 0 0" rpy="0 0 0" />
+                <geometry>
+                    <mesh filename="package://dagana_urdf/meshes/dg0001-simplified_v2.stl" scale="${mmTom} ${mmTom} ${mmTom}" />
+                </geometry>
+            </collision>
+        </xacro:if>
     </link>
     <joint name="${name}_claw_joint" type="${joint_type}">
@@ -41,27 +93,79 @@
     </joint>
     <link name="${name}_bottom_link">
-        <inertial>
-            <origin xyz="0 ${6.9644767e+01*mmTom} 0" rpy="0 0 0"/>
-            <mass value="4.6117745e-01"/>
-            <inertia iyy="${9.3855569e+02*mm2Tom2}"
-                     iyz="${-2.6445200e+02*mm2Tom2}"
-                     ixy="${7.1346830e+01*mm2Tom2}"
-                     izz="${1.9472731e+03*mm2Tom2}"
-                     ixz="${2.5290650e+00*mm2Tom2}"
-                     ixx="${1.4726991e+03*mm2Tom2}" />
-        </inertial>
-        <visual>
-            <origin xyz="0 0 0" rpy="0 0 0" />
-            <geometry>
-                <mesh filename="package://dagana_urdf/meshes/dg0002.stl" scale="${mmTom} ${mmTom} ${mmTom}" />
-            </geometry>
-            <material name="dagana_dark_grey"/>
-        </visual>
-        <collision>
-            <origin xyz="0 0 0" rpy="0 0 0" />
-            <geometry>
-                <mesh filename="package://dagana_urdf/meshes/dg0002-ch.stl" scale="${mmTom} ${mmTom} ${mmTom}" />
-            </geometry>
-        </collision>
+        <xacro:if value="${DAGANA_CLAWS_TYPE == 'centauro_claws'}">
+            <inertial>
+                <origin xyz="0 ${6.9644767e+01*mmTom} 0" rpy="0 0 0"/>
+                <mass value="4.6117745e-01"/>
+                <inertia iyy="${9.3855569e+02*mm2Tom2}"
+                        iyz="${-2.6445200e+02*mm2Tom2}"
+                        ixy="${7.1346830e+01*mm2Tom2}"
+                        izz="${1.9472731e+03*mm2Tom2}"
+                        ixz="${2.5290650e+00*mm2Tom2}"
+                        ixx="${1.4726991e+03*mm2Tom2}" />
+            </inertial>
+            <visual>
+                <origin xyz="0 0 0" rpy="0 0 0" />
+                <geometry>
+                    <mesh filename="package://dagana_urdf/meshes/dg0002.stl" scale="${mmTom} ${mmTom} ${mmTom}" />
+                </geometry>
+                <material name="dagana_dark_grey"/>
+            </visual>
+            <collision>
+                <origin xyz="0 0 0" rpy="0 0 0" />
+                <geometry>
+                    <mesh filename="package://dagana_urdf/meshes/dg0002-ch.stl" scale="${mmTom} ${mmTom} ${mmTom}" />
+                </geometry>
+            </collision>
+        </xacro:if>
+        <xacro:if value="${DAGANA_CLAWS_TYPE == 'concert_formwork_claws'}">
+            <inertial>
+                <origin xyz="0 ${6.9644767e+01*mmTom} 0" rpy="0 0 0"/>
+                <mass value="0.644"/>
+                <inertia iyy="${9.3855569e+02*mm2Tom2}"
+                        iyz="${-2.6445200e+02*mm2Tom2}"
+                        ixy="${7.1346830e+01*mm2Tom2}"
+                        izz="${1.9472731e+03*mm2Tom2}"
+                        ixz="${2.5290650e+00*mm2Tom2}"
+                        ixx="${1.4726991e+03*mm2Tom2}" />
+            </inertial>
+            <visual>
+                <origin xyz="0 0 0" rpy="0 0 0" />
+                <geometry>
+                    <mesh filename="package://dagana_urdf/meshes/dg0002.stl" scale="${mmTom} ${mmTom} ${mmTom}" />
+                </geometry>
+                <material name="dagana_dark_grey"/>
+            </visual>
+            <collision>
+                <origin xyz="0 0 0" rpy="0 0 0" />
+                <geometry>
+                    <mesh filename="package://dagana_urdf/meshes/dg0002-ch.stl" scale="${mmTom} ${mmTom} ${mmTom}" />
+                </geometry>
+            </collision>
+        </xacro:if>
+        <xacro:if value="${DAGANA_CLAWS_TYPE == 'concert_tube_claws'}">
+            <inertial>
+                <origin xyz="0 ${6.9644767e+01*mmTom} 0" rpy="0 0 0"/>
+                <mass value="0.608"/>
+                <inertia iyy="${9.3855569e+02*mm2Tom2}"
+                        iyz="${-2.6445200e+02*mm2Tom2}"
+                        ixy="${7.1346830e+01*mm2Tom2}"
+                        izz="${1.9472731e+03*mm2Tom2}"
+                        ixz="${2.5290650e+00*mm2Tom2}"
+                        ixx="${1.4726991e+03*mm2Tom2}" />
+            </inertial>
+            <visual>
+                <origin xyz="0 0 0" rpy="0 0 0" />
+                <geometry>
+                    <mesh filename="package://dagana_urdf/meshes/dg0002.stl" scale="${mmTom} ${mmTom} ${mmTom}" />
+                </geometry>
+                <material name="dagana_dark_grey"/>
+            </visual>
+            <collision>
+                <origin xyz="0 0 0" rpy="0 0 0" />
+                <geometry>
+                    <mesh filename="package://dagana_urdf/meshes/dg0002-ch.stl" scale="${mmTom} ${mmTom} ${mmTom}" />
+                </geometry>
+            </collision>
+        </xacro:if>
     </link>
     <!-- Manually put to have a transform in a "good" grasping spot-->

Commit message: add GAZEBO_URDF default param

File: dagana_urdf/urdf/config/dagana_config.urdf.xacro (robot description, xacro)
@@ -6,8 +6,8 @@
 <xacro:arg name="nicla_tof_visualize" default="true"/>
 <xacro:arg name="nicla_imu" default="true"/>
-<xacro:arg name="dagana_claws_type" default="centauro_claws"/>
 <!-- dagana_claws_types: - 'centauro_claws' -->
 <!--                     - 'concert_formwork_claws' -->
 <!--                     - 'concert_tube_claws'  -->
+<xacro:arg name="dagana_claws_type" default="centauro_claws"/>
 <xacro:property name="NICLA" value="$(arg nicla)" />
 <xacro:property name="NICLA_CAMERA" value="$(arg nicla_camera)" />

File: dagana_urdf/urdf/dagana_macro.urdf.xacro (robot description, xacro)
@@ -2,5 +2,5 @@
 <robot xmlns:xacro="http://ros.org/wiki/xacro">
 <xacro:include filename="$(find dagana_urdf)/urdf/config/dagana_config.urdf.xacro" />
-<xacro:macro name="dagana_gripper" params="name joint_type parent_link *origin">
+<xacro:macro name="dagana_gripper" params="name joint_type parent_link GAZEBO_URDF:=^|false *origin">
     <joint name="${name}_mount_joint" type="fixed">
         <xacro:insert_block name="origin"/>

Commit message: args for gazebo_urdf

File: dagana_urdf/urdf/config/dagana_config.urdf.xacro (robot description, xacro)
@@ -10,4 +10,5 @@
 <!--                     - 'concert_tube_claws'  -->
 <xacro:arg name="dagana_claws_type" default="centauro_claws"/>
+<xacro:arg name="gazebo_urdf" default="false"/>
 <xacro:property name="NICLA" value="$(arg nicla)" />
 <xacro:property name="NICLA_CAMERA" value="$(arg nicla_camera)" />
@@ -23,3 +24,4 @@
 <xacro:property name="PI" value="3.14159265359" />
 <xacro:property name="DAGANA_CLAWS_TYPE" value="$(arg dagana_claws_type)" />
+<xacro:property name="GAZEBO_URDF" value="$(arg gazebo_urdf)" />
 </robot>
