Commit message: different branches push caused mistake correction, add and test missing changes

File: dagana_urdf/urdf/config/dagana_config.urdf.xacro (robot description, xacro)
@@ -6,4 +6,9 @@
 <xacro:arg name="nicla_tof_visualize" default="true"/>
 <xacro:arg name="nicla_imu" default="true"/>
+<!-- dagana_claws_types: - 'centauro_claws' -->
+<!--                     - 'concert_formwork_claws' -->
+<!--                     - 'concert_tube_claws'  -->
+<xacro:arg name="dagana_claws_type" default="centauro_claws"/>
+<xacro:arg name="gazebo_urdf" default="false"/>
 <xacro:property name="NICLA" value="$(arg nicla)" />
 <xacro:property name="NICLA_CAMERA" value="$(arg nicla_camera)" />
@@ -18,3 +23,5 @@
 <xacro:property name="PI_2" value="1.57079632679" />
 <xacro:property name="PI" value="3.14159265359" />
+<xacro:property name="DAGANA_CLAWS_TYPE" value="$(arg dagana_claws_type)" />
+<xacro:property name="GAZEBO_URDF" value="$(arg gazebo_urdf)" />
 </robot>

File: dagana_urdf/urdf/dagana_macro.urdf.xacro (robot description, xacro)
@@ -2,5 +2,5 @@
 <robot xmlns:xacro="http://ros.org/wiki/xacro">
 <xacro:include filename="$(find dagana_urdf)/urdf/config/dagana_config.urdf.xacro" />
-<xacro:macro name="dagana_gripper" params="name joint_type parent_link *origin">
+<xacro:macro name="dagana_gripper" params="name joint_type parent_link GAZEBO_URDF:=^|false *origin">
     <joint name="${name}_mount_joint" type="fixed">
         <xacro:insert_block name="origin"/>
@@ -9,73 +9,413 @@
     </joint>
     <link name="${name}_top_link">
-        <inertial>
-            <origin xyz="${-6.3562154e+00*mmTom} ${-6.0265532e+00*mmTom}  ${6.0068288e+01*mmTom}" rpy="0 0 0"/>
-            <mass value="1.7432400"/>
-            <inertia ixx="${5.0510328e+03*mm2Tom2}"
-                     ixy="${-2.5264216e+02*mm2Tom2}"
-                     ixz="${-1.2103013e+02*mm2Tom2}"
-                     iyy="${4.7944612e+03*mm2Tom2}"
-                     iyz="${-7.3917704e+02*mm2Tom2}"
-                     izz="${3.1156997e+03*mm2Tom2}" />
-        </inertial>
-        <visual>
-            <origin xyz="0 0 0" rpy="0 0 0" />
-            <geometry>
-                <mesh filename="package://dagana_urdf/meshes/dg0001-simplified.stl" scale="${mmTom} ${mmTom} ${mmTom}" />
-            </geometry>
-            <material name="dagana_dark_grey"/>
-        </visual>
-        <collision>
-            <origin xyz="0 0 0" rpy="0 0 0" />
-            <geometry>
-                <mesh filename="package://dagana_urdf/meshes/dg0001-simplified_v2.stl" scale="${mmTom} ${mmTom} ${mmTom}" />
-            </geometry>
-        </collision>
+        <xacro:if value="${DAGANA_CLAWS_TYPE == 'centauro_claws'}">
+            <inertial>
+                <origin xyz="${-6.3562154e+00*mmTom} ${-6.0265532e+00*mmTom}  ${6.0068288e+01*mmTom}" rpy="0 0 0"/>
+                <mass value="1.7432400"/>
+                <inertia ixx="${5.0510328e+03*mm2Tom2}"
+                        ixy="${-2.5264216e+02*mm2Tom2}"
+                        ixz="${-1.2103013e+02*mm2Tom2}"
+                        iyy="${4.7944612e+03*mm2Tom2}"
+                        iyz="${-7.3917704e+02*mm2Tom2}"
+                        izz="${3.1156997e+03*mm2Tom2}" />
+            </inertial>
+            <visual>
+                <origin xyz="0 0 0" rpy="0 0 0" />
+                <geometry>
+                    <mesh filename="file://$(find dagana_urdf)/meshes/dg0001-simplified.stl" scale="${mmTom} ${mmTom} ${mmTom}" />
+                </geometry>
+                <material name="dagana_dark_grey"/>
+            </visual>
+            <collision>
+                <origin xyz="0 0 0" rpy="0 0 0" />
+                <geometry>
+                    <mesh filename="file://$(find dagana_urdf)/meshes/dg0001-simplified_v2.stl" scale="${mmTom} ${mmTom} ${mmTom}" />
+                </geometry>
+            </collision>
+        </xacro:if>
+        <xacro:if value="${DAGANA_CLAWS_TYPE == 'centauro_claws_palm_separated'}">
+            <!-- TODO this is the inertial of the entire piece (ABC), it should be divided among the different pieces -->
+            <inertial>
+                <origin xyz="${-6.3562154e+00*mmTom} ${-6.0265532e+00*mmTom}  ${6.0068288e+01*mmTom}" rpy="0 0 0"/>
+                <mass value="1.7432400"/>
+                <inertia ixx="${5.0510328e+03*mm2Tom2}"
+                        ixy="${-2.5264216e+02*mm2Tom2}"
+                        ixz="${-1.2103013e+02*mm2Tom2}"
+                        iyy="${4.7944612e+03*mm2Tom2}"
+                        iyz="${-7.3917704e+02*mm2Tom2}"
+                        izz="${3.1156997e+03*mm2Tom2}" />
+            </inertial>
+            <visual>
+                <origin xyz="0 0 0" rpy="0 0 0" />
+                <geometry>
+                    <mesh filename="file://$(find dagana_urdf)/meshes/dagana_fixed_A.stl" scale="${mmTom} ${mmTom} ${mmTom}" />
+                </geometry>
+                <material name="dagana_dark_grey"/>
+            </visual>
+            <collision>
+                <origin xyz="0 0 0" rpy="0 0 0" />
+                <geometry>
+                    <mesh filename="file://$(find dagana_urdf)/meshes/dagana_fixed_A_simple.stl" scale="${mmTom} ${mmTom} ${mmTom}" />
+                </geometry>
+            </collision>
+        </xacro:if>
+        <xacro:if value="${DAGANA_CLAWS_TYPE == 'concert_formwork_claws' or DAGANA_CLAWS_TYPE == 'concert_tube_claws'}">
+            <inertial>
+                <origin xyz="${-6.2068321e+00*mmTom} ${-1.1480379e+01*mmTom}  ${4.7628197e+01*mmTom}" rpy="0 0 0"/>
+                <mass value="1.548"/>
+                <inertia ixx="${2.8611741e+03*mm2Tom2}"
+                        ixy="${-2.7536524e+00*mm2Tom2}"
+                        ixz="${-1.8353431e+02*mm2Tom2}"
+                        iyy="${2.5520008e+03*mm2Tom2}"
+                        iyz="${1.1763870e+02*mm2Tom2}"
+                        izz="${3.0966827e+03*mm2Tom2}" />
+            </inertial>
+            <visual>
+                <origin xyz="0 0 0" rpy="0 0 0" />
+                <geometry>
+                    <mesh filename="file://$(find dagana_urdf)/meshes/mesh_dagana-base_simple.stl" scale="${mmTom} ${mmTom} ${mmTom}" />
+                </geometry>
+                <material name="dagana_dark_grey"/>
+            </visual>
+            <collision>
+                <origin xyz="0 0 0" rpy="0 0 0" />
+                <geometry>
+                    <mesh filename="file://$(find dagana_urdf)/meshes/mesh_dagana-base_ch.stl" scale="${mmTom} ${mmTom} ${mmTom}" />
+                </geometry>
+            </collision>
+        </xacro:if>
     </link>
-    <joint name="${name}_claw_joint" type="${joint_type}">
-        <origin xyz="${0.0*mmTom} ${-28.00*mmTom} ${50.25*mmTom}" rpy="${PI_2} 0 ${PI}"/>
-        <parent link="${name}_top_link"/>
-        <child link="${name}_bottom_link"/>
-        <axis xyz="-1 0 0"/>
-        <limit effort="1000" lower="0" upper="1.3" velocity="10.0"/>
-    </joint>
+    <xacro:if value="${DAGANA_CLAWS_TYPE == 'centauro_claws_palm_separated'}">
+        <joint name="${name}_fixed_A_B_fixed_joint" type="fixed" dont_collapse="true">
+            <origin xyz="0 0 0" rpy="0 0 0"/>
+            <parent link="${name}_top_link"/>
+            <child link="${name}_fixed_B"/>
+        </joint>
+        <link name="${name}_fixed_B">
+            <visual>
+                <origin xyz="0 0 0" rpy="0 0 0" />
+                <geometry>
+                    <mesh filename="file://$(find dagana_urdf)/meshes/dagana_fixed_B.stl" scale="${mmTom} ${mmTom} ${mmTom}" />
+                </geometry>
+                <material name="dagana_dark_grey"/>
+            </visual>
+            <collision>
+                <origin xyz="0 0 0" rpy="0 0 0" />
+                <geometry>
+                    <mesh filename="file://$(find dagana_urdf)/meshes/dagana_fixed_B_simple.stl" scale="${mmTom} ${mmTom} ${mmTom}" />
+                </geometry>
+            </collision>
+        </link>
+        <joint name="${name}_fixed_B_C_fixed_joint" type="fixed" dont_collapse="true">
+            <origin xyz="0 0 0" rpy="0 0 0"/>
+            <parent link="${name}_fixed_B"/>
+            <child link="${name}_fixed_C"/>
+        </joint>
+        <link name="${name}_fixed_C">
+            <visual>
+                <origin xyz="0 0 0" rpy="0 0 0" />
+                <geometry>
+                    <mesh filename="file://$(find dagana_urdf)/meshes/dagana_fixed_C.stl" scale="${mmTom} ${mmTom} ${mmTom}" />
+                </geometry>
+                <material name="dagana_dark_grey"/>
+            </visual>
+            <collision>
+                <origin xyz="0 0 0" rpy="0 0 0" />
+                <geometry>
+                    <mesh filename="file://$(find dagana_urdf)/meshes/dagana_fixed_C_simple.stl" scale="${mmTom} ${mmTom} ${mmTom}" />
+                </geometry>
+            </collision>
+        </link>
+    </xacro:if>
+    <xacro:if value="${DAGANA_CLAWS_TYPE == 'concert_formwork_claws' or DAGANA_CLAWS_TYPE == 'concert_tube_claws'}">
+        <joint name="${name}_claw_joint" type="${joint_type}">
+            <origin xyz="${0.0*mmTom} ${-28.00*mmTom} ${50.25*mmTom}" rpy="${-PI} ${-PI_2} 0 "/>
+            <parent link="${name}_top_link"/>
+            <child link="${name}_bottom_link"/>
+            <axis xyz="0 0 1"/>
+            <limit effort="1000" lower="-1.5" upper="1.3" velocity="10.0"/>
+        </joint>
+    </xacro:if>
+    <xacro:if value="${DAGANA_CLAWS_TYPE == 'centauro_claws' or DAGANA_CLAWS_TYPE == 'centauro_claws_palm_separated'}">
+        <joint name="${name}_claw_joint" type="${joint_type}">
+            <origin xyz="${0.0*mmTom} ${-28.00*mmTom} ${50.25*mmTom}" rpy="${PI_2} 0 ${PI}"/>
+            <parent link="${name}_top_link"/>
+            <child link="${name}_bottom_link"/>
+            <axis xyz="-1 0 0"/>
+            <limit effort="1000" lower="-0.1" upper="1.3" velocity="10.0"/>
+        </joint>
+    </xacro:if>
     <link name="${name}_bottom_link">
-        <inertial>
-            <origin xyz="0 ${6.9644767e+01*mmTom} 0" rpy="0 0 0"/>
-            <mass value="4.6117745e-01"/>
-            <inertia iyy="${9.3855569e+02*mm2Tom2}"
-                     iyz="${-2.6445200e+02*mm2Tom2}"
-                     ixy="${7.1346830e+01*mm2Tom2}"
-                     izz="${1.9472731e+03*mm2Tom2}"
-                     ixz="${2.5290650e+00*mm2Tom2}"
-                     ixx="${1.4726991e+03*mm2Tom2}" />
-        </inertial>
-        <visual>
-            <origin xyz="0 0 0" rpy="0 0 0" />
-            <geometry>
-                <mesh filename="package://dagana_urdf/meshes/dg0002.stl" scale="${mmTom} ${mmTom} ${mmTom}" />
-            </geometry>
-            <material name="dagana_dark_grey"/>
-        </visual>
-        <collision>
-            <origin xyz="0 0 0" rpy="0 0 0" />
-            <geometry>
-                <mesh filename="package://dagana_urdf/meshes/dg0002-ch.stl" scale="${mmTom} ${mmTom} ${mmTom}" />
-            </geometry>
-        </collision>
+        <xacro:if value="${DAGANA_CLAWS_TYPE == 'centauro_claws'}">
+            <inertial>
+                <origin xyz="0 ${6.9644767e+01*mmTom} 0" rpy="0 0 0"/>
+                <mass value="4.6117745e-01"/>
+                <inertia iyy="${9.3855569e+02*mm2Tom2}"
+                        iyz="${-2.6445200e+02*mm2Tom2}"
+                        ixy="${7.1346830e+01*mm2Tom2}"
+                        izz="${1.9472731e+03*mm2Tom2}"
+                        ixz="${2.5290650e+00*mm2Tom2}"
+                        ixx="${1.4726991e+03*mm2Tom2}" />
+            </inertial>
+            <visual>
+                <origin xyz="0 0 0" rpy="0 0 0" />
+                <geometry>
+                    <mesh filename="file://$(find dagana_urdf)/meshes/dg0002.stl" scale="${mmTom} ${mmTom} ${mmTom}" />
+                </geometry>
+                <material name="dagana_dark_grey"/>
+            </visual>
+            <collision>
+                <origin xyz="0 0 0" rpy="0 0 0" />
+                <geometry>
+                    <mesh filename="file://$(find dagana_urdf)/meshes/dg0002-ch.stl" scale="${mmTom} ${mmTom} ${mmTom}" />
+                </geometry>
+            </collision>
+        </xacro:if>
+        <xacro:if value="${DAGANA_CLAWS_TYPE == 'centauro_claws_palm_separated'}">
+            <inertial>
+                <origin xyz="0 ${6.9644767e+01*mmTom} 0" rpy="0 0 0"/>
+                <mass value="4.6117745e-01"/>
+                <inertia iyy="${9.3855569e+02*mm2Tom2}"
+                        iyz="${-2.6445200e+02*mm2Tom2}"
+                        ixy="${7.1346830e+01*mm2Tom2}"
+                        izz="${1.9472731e+03*mm2Tom2}"
+                        ixz="${2.5290650e+00*mm2Tom2}"
+                        ixx="${1.4726991e+03*mm2Tom2}" />
+            </inertial>
+            <visual>
+                <origin xyz="0 0 0" rpy="0 0 0" />
+                <geometry>
+                    <mesh filename="file://$(find dagana_urdf)/meshes/dagana_claw_A.stl" scale="${mmTom} ${mmTom} ${mmTom}" />
+                </geometry>
+                <material name="dagana_dark_grey"/>
+            </visual>
+            <collision>
+                <origin xyz="0 0 0" rpy="0 0 0" />
+                <geometry>
+                    <mesh filename="file://$(find dagana_urdf)/meshes/dagana_claw_A_simple.stl" scale="${mmTom} ${mmTom} ${mmTom}" />
+                </geometry>
+            </collision>
+        </xacro:if>
+        <xacro:if value="${DAGANA_CLAWS_TYPE == 'concert_formwork_claws' or DAGANA_CLAWS_TYPE == 'concert_tube_claws'}">
+            <inertial>
+                <origin xyz="${2.5812008e+01*mmTom} ${2.5751001e+00*mmTom} ${-4.9454259e+00*mmTom}" rpy="0 0 0"/>
+                <mass value="2.18e-01"/>
+                <inertia ixx="${4.5712825e+02*mm2Tom2}"
+                        ixy="${-1.1939252e+01*mm2Tom2}"
+                        ixz="${-3.2916995e+01*mm2Tom2}"
+                        iyy="${5.3267788e+02*mm2Tom2}"
+                        iyz="${-2.1469634e+00*mm2Tom2}"
+                        izz="${1.5156084e+02*mm2Tom2}"/>
+            </inertial>
+            <visual>
+                <origin xyz="0 0 0" rpy="0 0 0" />
+                <geometry>
+                    <mesh filename="file://$(find dagana_urdf)/meshes/mesh_dagana-link_simple.stl" scale="${mmTom} ${mmTom} ${mmTom}" />
+                </geometry>
+                <material name="dagana_dark_grey"/>
+            </visual>
+            <collision>
+                <origin xyz="0 0 0" rpy="0 0 0" />
+                <geometry>
+                    <mesh filename="file://$(find dagana_urdf)/meshes/mesh_dagana-link_ch.stl" scale="${mmTom} ${mmTom} ${mmTom}" />
+                </geometry>
+            </collision>
+        </xacro:if>
     </link>
-    <!-- Manually put to have a transform in a "good" grasping spot-->
+    <xacro:if value="${DAGANA_CLAWS_TYPE == 'centauro_claws_palm_separated'}">
+        <joint name="${name}_claw_A_B_fixed_joint" type="fixed" dont_collapse="true">
+            <origin xyz="0 0 0" rpy="0 0 0"/>
+            <parent link="${name}_bottom_link"/>
+            <child link="${name}_claw_B"/>
+        </joint>
+        <link name="${name}_claw_B">
+            <visual>
+                <origin xyz="0 0 0" rpy="0 0 0" />
+                <geometry>
+                    <mesh filename="file://$(find dagana_urdf)/meshes/dagana_claw_B.stl" scale="${mmTom} ${mmTom} ${mmTom}" />
+                </geometry>
+                <material name="dagana_dark_grey"/>
+            </visual>
+            <collision>
+                <origin xyz="0 0 0" rpy="0 0 0" />
+                <geometry>
+                    <mesh filename="file://$(find dagana_urdf)/meshes/dagana_claw_B_simple.stl" scale="${mmTom} ${mmTom} ${mmTom}" />
+                </geometry>
+            </collision>
+        </link>
+    </xacro:if>
+    <xacro:if value="${GAZEBO_URDF}">
+        <gazebo reference="${name}_bottom_link">
+            <mu1>1</mu1>
+            <mu2>1</mu2>
+            <kp>100000.0</kp>
+            <kd>1.0</kd>
+            <maxVel>0.0</maxVel>
+            <minDepth>0.0001</minDepth>
+            <selfCollide>True</selfCollide>
+            <material>Gazebo/DarkGrey</material>
+        </gazebo>
+        <gazebo reference="${name}_top_link">
+            <mu1>1</mu1>
+            <mu2>1</mu2>
+            <kp>100000.0</kp>
+            <kd>1.0</kd>
+            <maxVel>0.0</maxVel>
+            <minDepth>0.0001</minDepth>
+            <selfCollide>True</selfCollide>
+            <material>Gazebo/DarkGrey</material>
+        </gazebo>
+    </xacro:if>
+    <!-- TCP frame: Manually put to have a transform in a "good" grasping spot-->
     <joint name="${name}_tcp_joint" type="fixed">
-        <origin xyz="0 -0.05 0.15" rpy="0 0 0"/>
+        <xacro:if value="${DAGANA_CLAWS_TYPE == 'centauro_claws'}">
+            <origin xyz="0 -0.04 0.16" rpy="0 0 0"/>
+        </xacro:if>
+        <xacro:if value="${DAGANA_CLAWS_TYPE == 'concert_formwork_claws' or DAGANA_CLAWS_TYPE == 'concert_tube_claws'}">
+            <origin xyz="0 -0.05 0.18" rpy="0 0 0"/>
+        </xacro:if>
         <parent link="${name}_top_link"/>
         <child link="${name}_tcp"/>
     </joint>
     <link name="${name}_tcp"></link>
-    <gazebo reference="${name}_bottom_link">
-        <material>Gazebo/DarkGrey</material>
-    </gazebo>
-    <gazebo reference="${name}_top_link">
-        <material>Gazebo/DarkGrey</material>
-    </gazebo>
+    <!-- Dagana Jaws : Formwork / Tube -->
+    <xacro:if value="${DAGANA_CLAWS_TYPE == 'concert_formwork_claws'}">
+        <link name="${name}_bottom_link_jaw">
+            <inertial>
+                <origin xyz="0.0 ${-5.0362316e+00*mmTom} ${4.8400486e+01*mmTom}" rpy="0 0 0"/>
+                <mass value="4.26e-01"/>
+                <inertia ixx="${5.6823263e+02*mm2Tom2}"
+                        ixy="${0.0*mm2Tom2}"
+                        ixz="${0.0*mm2Tom2}"
+                        iyy="${9.3524040e+02*mm2Tom2}"
+                        iyz="${5.2302782e+01*mm2Tom2}"
+                        izz="${5.0082202e+02*mm2Tom2}"/>
+            </inertial>
+            <visual>
+                <origin xyz="0 0 0" rpy="0 0 0" />
+                <geometry>
+                    <mesh filename="file://$(find dagana_urdf)/meshes/mesh_formwork-base.stl" scale="${mmTom} ${mmTom} ${mmTom}" />
+                </geometry>
+                <material name="dagana_dark_grey"/>
+            </visual>
+            <collision>
+                <origin xyz="0 0 0" rpy="0 0 0" />
+                <geometry>
+                    <mesh filename="file://$(find dagana_urdf)/meshes/mesh_formwork-base_ch.stl" scale="${mmTom} ${mmTom} ${mmTom}" />
+                </geometry>
+            </collision>
+        </link>
+        <link name="${name}_top_link_jaw">
+            <inertial>
+                <origin xyz="0.0 ${-3.3025449e+00*mmTom} ${5.2167268e+01*mmTom}" rpy="0 0 0"/>
+                <mass value="3.52e-01"/>
+                <inertia ixx="${5.2459269e+02*mm2Tom2}"
+                        ixy="${0.0*mm2Tom2}"
+                        ixz="${0.0*mm2Tom2}"
+                        iyy="${8.5587829e+02*mm2Tom2}"
+                        iyz="${6.0052568e+01*mm2Tom2}"
+                        izz="${4.4262897e+02*mm2Tom2}"/>
+            </inertial>
+            <visual>
+                <origin xyz="0 0 0" rpy="0 0 0" />
+                <geometry>
+                    <mesh filename="file://$(find dagana_urdf)/meshes/mesh_formwork-thumb.stl" scale="${mmTom} ${mmTom} ${mmTom}" />
+                </geometry>
+                <material name="dagana_dark_grey"/>
+            </visual>
+            <collision>
+                <origin xyz="0 0 0" rpy="0 0 0" />
+                <geometry>
+                    <mesh filename="file://$(find dagana_urdf)/meshes/mesh_formwork-thumb_ch.stl" scale="${mmTom} ${mmTom} ${mmTom}" />
+                </geometry>
+            </collision>
+        </link>
+    </xacro:if>
+    <xacro:if value="${DAGANA_CLAWS_TYPE == 'concert_tube_claws'}">
+        <link name="${name}_bottom_link_jaw">
+            <inertial>
+                <origin xyz="0.0 ${3.5142417e+00*mmTom} ${5.6108761e+01*mmTom}" rpy="0 0 0"/>
+                <mass value="3.7384233e-01"/>
+                <inertia ixx="${8.3782493e+02*mm2Tom2}"
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
Commit message: inline material definition to avoid duplication (leads to gz crash)

File: dagana_urdf/urdf/config/dagana_config.urdf.xacro (robot description, xacro)
@@ -16,7 +16,4 @@
 <xacro:property name="nicla_tof_visualize" value="$(arg nicla_tof_visualize)" />
 <xacro:property name="NICLA_IMU" value="$(arg nicla_imu)" />
-<material name="dagana_dark_grey">
-	<color rgba="0.2 0.2 0.2 1"/>
-</material>
 <xacro:property name="mmTom" value="1e-3" />
 <xacro:property name="mm2Tom2" value="1e-6" />

File: dagana_urdf/urdf/dagana_macro.urdf.xacro (robot description, xacro)
@@ -3,4 +3,7 @@
 <xacro:include filename="$(find dagana_urdf)/urdf/config/dagana_config.urdf.xacro" />
 <xacro:macro name="dagana_gripper" params="name joint_type parent_link GAZEBO_URDF:=^|false *origin">
+    <material name="dagana_dark_grey_${name}">
+        <color rgba="0.2 0.2 0.2 1"/>
+    </material>
     <joint name="${name}_mount_joint" type="fixed">
         <xacro:insert_block name="origin"/>
